Commit message: Automated update by GitHub Action

File: urdfrobot.urdf (robot description, URDF)
Before this commit: robot rover, 14 links, 13 joints
Joints:
- joint l3_l4: origin xyz=0.1524 0 -0.0508 rpy=0 -1.5708 0 -> xyz=0.1524 -0 -0.0508 rpy=-0 -1.5708 0
- joint l4_l5: origin xyz=0.0508 0 -0.2032 rpy=3.14159 1.5708 0 -> xyz=0.0508 -0 -0.2032 rpy=-3.14159 1.5708 0
