Commit message: Automated update by GitHub Action

File: RescueRangersArm.urdf (robot description, URDF)
Before this commit: robot rescue_rangers_arm, 7 links, 6 joints
Links:
- link frame: mass 1e-09 -> 0.183726
Joints:
- joint j4: origin xyz=-0.045 -0 -0.027 rpy=-0 1.5708 0 -> xyz=-0.045 -0 -0.027 rpy=0 1.5708 0
- joint j5: origin xyz=0.045 3.91302e-05 -0.027 rpy=0 -1.5708 0 -> xyz=0.045 3.91302e-05 -0.027 rpy=-0 -1.5708 0
