Commit message: mess with cmake to make meshes save to correct dir

File: urdf/RescueRangersArm.urdf (robot description, URDF)
Before this commit: robot rescue_rangers_arm, 7 links, 6 joints
Links:
- link frame: geometry collision mesh filename=package://rover_description/share/rover_description/RescueR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; collision mesh filename=package://rover_description/share/rover_description/RescueR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
- link h42p_020_s300_r_dummy2: geometry collision mesh filename=package://rover_description/share/rover_description/RescueR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; collision mesh filename=package://rover_description/share/rover_description/RescueR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
- link h42p_020_s300_r_dummy2_2: geometry collision mesh filename=package://rover_description/share/rover_description/RescueR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; collision mesh filename=package://rover_description/share/rover_description/RescueR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
- link j3: geometry collision mesh filename=package://rover_description/share/rover_description/RescueR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; collision mesh filename=package://rover_description/share/rover_description/RescueR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
- link j5: geometry collision mesh filename=package://rover_description/share/rover_description/RescueR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; collision mesh filename=package://rover_description/share/rover_description/RescueR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
- link part_5: geometry collision mesh filename=package://rover_description/share/rover_description/RescueR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; collision mesh filename=package://rover_description/share/rover_description/RescueR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
- link part_5_2: geometry collision mesh filename=package://rover_description/share/rover_description/RescueR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; collision mesh filename=package://rover_description/share/rover_description/RescueR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
